File: exynos-backpack.sch (EAGLE design)
At the start: 56 parts, among them IC1 MIC5335-SPYMT, IC2 TXS0108ERGY, IC3 LTC4352DD, IC4 LTC4352DD, IC5 LTC4352DD, J1 POWER_JACKPTH_LOCK, Q1 SI7234DP, Q2 SI7234DP, Q3 SI7234DP

Commit message: More work on backpack placement
Parts:
- removed C1, C2, C3, C4, C5, C6: 0.1uF, biomimetic:CAP0402-CAP
- removed C7, C8, C9: 22uF, biomimetic:CAP0603-CAP
- removed D1, D2, D3: PESD5V0S1UA, biomimetic:PESD5V0S1UA
- removed IC3, IC4, IC5: LTC4352DD, biomimetic:LTC4352DD
- removed J1: POWER_JACKPTH_LOCK, biomimetic:POWER_JACKPTH_LOCK
- removed JP5, JP6: JST-RCY-MALE, biomimetic:JST-RCY-MALE
- removed LED1, LED3, LED5: FAULT_BATTA, biomimetic:LED0603
- removed LED2, LED4, LED6: STATUS_BATTA, biomimetic:LED0603
- removed Q1, Q2, Q3: SI7234DP, biomimetic:SI7234DP
- removed R1, R11: 1.5k, biomimetic:RESISTOR0402-RES
- removed R10, R9: 510, biomimetic:RESISTOR0402-RES
- removed R12, R2: 20k, biomimetic:RESISTOR0402-RES
- removed R13, R3, R8: 2.7k, biomimetic:RESISTOR0402-RES
- removed R14, R15, R4, R5: 330, biomimetic:RESISTOR0402-RES
- removed R6: 910, biomimetic:RESISTOR0402-RES
- removed R7: 27k, biomimetic:RESISTOR0402-RES
- added JP3: JST-RCY-MALE, biomimetic:JST-RCY-MALE
Connections:
- removed net N$1: C1.2, IC3.SOURCE, Q1A.S, Q1B.S
- removed net N$10: IC3.!STATUS, LED2.C
- removed net N$11: LED2.A, R5.1
- removed net N$12: LED1.A, R4.1
- removed net N$13: C3.2, IC5.SOURCE, Q2A.S, Q2B.S
- removed net N$14: IC5.GATE, Q2A.G, Q2B.G
- removed net N$15: C3.1, IC5.CPO
- removed net N$18: IC5.UV, R6.2, R7.1
- removed net N$19: IC5.OV, R6.1, R8.2
- removed net N$2: IC3.GATE, Q1A.G, Q1B.G
- removed net N$20: C4.1, IC5.VCC
- removed net N$21: IC5.!FAULT, LED3.C
- removed net N$22: IC5.!STATUS, LED4.C
- removed net N$23: LED4.A, R10.1
- removed net N$24: LED3.A, R9.1
- removed net N$25: C5.2, IC4.SOURCE, Q3A.S, Q3B.S
- removed net N$26: IC4.GATE, Q3A.G, Q3B.G
- removed net N$27: C5.1, IC4.CPO
- removed net N$30: IC4.UV, R11.2, R12.1
- removed net N$31: IC4.OV, R11.1, R13.2
- removed net N$32: C6.1, IC4.VCC
- removed net N$33: IC4.!FAULT, LED5.C
- removed net N$34: IC4.!STATUS, LED6.C
- removed net N$35: LED6.A, R15.1
- removed net N$36: LED5.A, R14.1
- removed net N$4: C1.1, IC3.CPO
- removed net N$6: IC3.UV, R1.2, R2.1
- removed net N$7: IC3.OV, R1.1, R3.2
- removed net N$8: C2.1, IC3.VCC
- removed net N$9: IC3.!FAULT, LED1.C
- removed net V_BATTA: C7.1, D1.C, IC3.VIN, Q1A.D, R2.2, R4.2, R5.2
- removed net V_BATTB: C8.1, D2.C, IC4.VIN, Q3A.D, R12.2, R14.2, R15.2
- removed net V_WALL: C9.1, D3.C, IC5.VIN, Q2A.D, R10.2, R7.2, R9.2
- net GND: no longer C2.2, C4.2, C6.2, C7.2, C8.2, C9.2, D1.A, D2.A, D3.A, IC3.GND, IC3.REV, IC4.GND, IC4.REV, IC5.GND, IC5.REV, R13.1, R3.1, R8.1
- net V_OR: no longer IC3.OUT, IC4.OUT, IC5.OUT, Q1B.D, Q2B.D, Q3B.D
Other:
- moved on the sheet: C15, C16, IC2, JP1, JP2

Commit message: First pass at exynos backpack placement
Parts:
- removed JP7: JST-RCY-MALE, biomimetic:JST-RCY-MALE
- IC2: value TXS0108ERGY -> TXB0108RGY; device biomimetic:TXS0108ERGY -> biomimetic:TXB0108RGY
- JP1: value CONSOLE -> (none); device biomimetic:MOLEX_503480-0600 -> biomimetic:M04MOLEX_5267
Connections:
- removed net UART_RX_1V8: IC2.A2, JP1.4
- removed net UART_RX_3V3: IC2.B2, JP2.4
- removed net UART_TX_1V8: IC2.A1, JP1.5
- removed net UART_TX_3V3: IC2.B1, JP2.6
- removed net V_OR: C10.1, PS1.VIN
- new net IMAGEPROC_RXD: IC2.B2
- new net IMAGEPROC_TXD: IC2.B3
- new net ODROID_RXD: IC2.A3, JP1.3
- new net ODROID_TXD: IC2.A2, JP1.2
- net 1.8V: now also IC2.A1, JP1.1
- net 3.3V: now also IC2.B1
- net GND: now also IC2.A4, IC2.A5, IC2.A6, IC2.A7, IC2.A8, IC2.B4, IC2.B5, IC2.B6, IC2.B7, IC2.B8, JP1.4, JP3.1; no longer JP1.1, JP2.3, JP2.5
- net V_BATT: now also C10.1, JP3.2, PS1.VIN; no longer JP2.1, JP2.2

Commit message: Finish placement
Parts:
- added JP4: JST-RCY-FEMALE-NOSILK, biomimetic:JST-RCY-FEMALE-NOSILK
- added JP5: ODROID CONSOLE, biomimetic:M04MOLEX_5267
- JP1: value (none) -> ODROID
- JP3: value JST-RCY-MALE -> JST-RCY-MALE-NOSILK; device biomimetic:JST-RCY-MALE -> biomimetic:JST-RCY-MALE-NOSILK
Connections:
- net 1.8V: now also JP5.1; no longer IC2.A1
- net 3.3V: no longer IC2.B1
- net 5V: now also JP4.2
- net GND: now also IC2.A1, IC2.B1, JP2.3, JP2.5, JP4.1, JP5.4
- net IMAGEPROC_RXD: now also JP2.6
- net IMAGEPROC_TXD: now also JP2.4
- net ODROID_RXD: now also JP5.3
- net ODROID_TXD: now also JP5.2
Other:
- note added: "Boost Converter"
- note added: "Level Translator"
