File: exynos-backpack.sch (EAGLE design)
At the start: 16 parts, among them IC1 MIC5335-SPYMT, IC2 TXB0108RGY

Commit message: Arrange silkscreen
Parts:
- removed C14: 1uF, biomimetic:CAP0402-CAP
- JP1: value ODROID -> ODROID UART; device biomimetic:M04MOLEX_5267 -> biomimetic:M041X04_MOLEX_5267_NOSILK
- JP3: value JST-RCY-MALE-NOSILK -> BATTERY
- JP4: value JST-RCY-FEMALE-NOSILK -> ODROID 5V
- JP5: value ODROID CONSOLE -> CONSOLE
Connections:
- removed net 3.0V: C14.1, IC1.3.0
- net GND: now also IC1.EN_3.0V; no longer C14.2
- net V_BATT: no longer IC1.EN_3.0V
Other:
- moved on the sheet: C13
Changed lines of the file:
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@@
 <part name="C12" library="biomimetic" deviceset="CAP" device="0402-CAP" value="1uF"/>
 <part name="C13" library="biomimetic" deviceset="CAP" device="0402-CAP" value="1uF"/>
-<part name="C14" library="biomimetic" deviceset="CAP" device="0402-CAP" value="1uF"/>
 <part name="U$4" library="biomimetic" deviceset="V_BATT" device=""/>
 <part name="GND9" library="biomimetic" deviceset="GND" device=""/>
 <part name="P+1" library="biomimetic" deviceset="3.3V" device=""/>
-<part name="U$5" library="biomimetic" deviceset="3.0V" device=""/>
 <part name="GND10" library="biomimetic" deviceset="GND" device=""/>
-<part name="GND11" library="biomimetic" deviceset="GND" device=""/>
 <part name="IC2" library="biomimetic" deviceset="TXB0108" device="RGY"/>
 <part name="U$10" library="biomimetic" deviceset="1.8V" device=""/>
@@
 <part name="GND23" library="biomimetic" deviceset="GND" device=""/>
 <part name="U$2" library="biomimetic" deviceset="ODROID-U2" device=""/>
-<part name="JP3" library="biomimetic" deviceset="JST-RCY-MALE" device="-NOSILK" value="JST-RCY-MALE-NOSILK"/>
+<part name="JP3" library="biomimetic" deviceset="JST-RCY-MALE" device="-NOSILK" value="BATTERY"/>
 <part name="U$3" library="biomimetic" deviceset="1.8V" device=""/>
 <part name="GND1" library="biomimetic" deviceset="GND" device=""/>
 <part name="GND2" library="biomimetic" deviceset="GND" device=""/>
 <part name="GND3" library="biomimetic" deviceset="GND" device=""/>
-<part name="JP1" library="biomimetic" deviceset="M04" device="MOLEX_5267" value="ODROID"/>
+<part name="JP1" library="biomimetic" deviceset="M04" device="1X04_MOLEX_5267_NOSILK" value="ODROID UART"/>
 <part name="GND4" library="biomimetic" deviceset="GND" device=""/>
-<part name="JP4" library="biomimetic" deviceset="JST-RCY-FEMALE" device="-NOSILK"/>
+<part name="JP4" library="biomimetic" deviceset="JST-RCY-FEMALE" device="-NOSILK" value="ODROID 5V"/>
 <part name="P+3" library="biomimetic" deviceset="3.3V" device=""/>
 <part name="U$6" library="biomimetic" deviceset="1.8V" device=""/>
@@
 <part name="U$13" library="biomimetic" deviceset="1.8V" device=""/>
 <part name="GND7" library="biomimetic" deviceset="GND" device=""/>
-<part name="JP5" library="biomimetic" deviceset="M04" device="MOLEX_5267" value="ODROID CONSOLE"/>
+<part name="JP5" library="biomimetic" deviceset="M04" device="MOLEX_5267" value="CONSOLE"/>
 </parts>
 <sheets>
@@
 <instance part="IC1" gate="G$1" x="35.56" y="30.48"/>
 <instance part="C12" gate="G$1" x="15.24" y="30.48" rot="R180"/>
-<instance part="C13" gate="G$1" x="55.88" y="40.64"/>
-<instance part="C14" gate="G$1" x="55.88" y="12.7"/>
+<instance part="C13" gate="G$1" x="55.88" y="27.94"/>
 <instance part="U$4" gate="G$1" x="15.24" y="48.26"/>
 <instance part="GND9" gate="1" x="15.24" y="17.78"/>
-<instance part="P+1" gate="G$1" x="55.88" y="48.26"/>
-<instance part="U$5" gate="G$1" x="55.88" y="20.32"/>
-<instance part="GND10" gate="1" x="55.88" y="33.02"/>
-<instance part="GND11" gate="1" x="55.88" y="5.08"/>
+<instance part="P+1" gate="G$1" x="55.88" y="35.56"/>
+<instance part="GND10" gate="1" x="55.88" y="20.32"/>
 <instance part="IC2" gate="G$1" x="121.92" y="114.3"/>
 <instance part="U$10" gate="G$1" x="119.38" y="137.16" smashed="yes">
@@
 <pinref part="IC1" gate="G$1" pin="GND"/>
 <wire x1="15.24" y1="22.86" x2="15.24" y2="20.32" width="0.1524" layer="91"/>
-<wire x1="22.86" y1="22.86" x2="15.24" y2="22.86" width="0.1524" layer="91"/>
+<wire x1="22.86" y1="22.86" x2="20.32" y2="22.86" width="0.1524" layer="91"/>
 <junction x="15.24" y="22.86"/>
+<pinref part="IC1" gate="G$1" pin="EN_3.0V"/>
+<wire x1="20.32" y1="22.86" x2="15.24" y2="22.86" width="0.1524" layer="91"/>
+<wire x1="22.86" y1="27.94" x2="20.32" y2="27.94" width="0.1524" layer="91"/>
+<wire x1="20.32" y1="27.94" x2="20.32" y2="22.86" width="0.1524" layer="91"/>
+<junction x="20.32" y="22.86"/>
 </segment>
 <segment>
 <pinref part="GND10" gate="1" pin="GND"/>
 <pinref part="C13" gate="G$1" pin="2"/>
-<wire x1="55.88" y1="35.56" x2="55.88" y2="38.1" width="0.1524" layer="91"/>
-</segment>
-<segment>
-<pinref part="C14" gate="G$1" pin="2"/>
-<pinref part="GND11" gate="1" pin="GND"/>
-<wire x1="55.88" y1="10.16" x2="55.88" y2="7.62" width="0.1524" layer="91"/>
+<wire x1="55.88" y1="22.86" x2="55.88" y2="25.4" width="0.1524" layer="91"/>
 </segment>
 <segment>
@@
 <pinref part="U$4" gate="G$1" pin="V_BATT"/>
 <wire x1="15.24" y1="33.02" x2="15.24" y2="38.1" width="0.1524" layer="91"/>
-<pinref part="IC1" gate="G$1" pin="EN_3.0V"/>
 <wire x1="15.24" y1="38.1" x2="15.24" y2="48.26" width="0.1524" layer="91"/>
-<wire x1="22.86" y1="27.94" x2="20.32" y2="27.94" width="0.1524" layer="91"/>
-<wire x1="20.32" y1="27.94" x2="20.32" y2="33.02" width="0.1524" layer="91"/>
 <pinref part="IC1" gate="G$1" pin="VIN"/>
 <wire x1="20.32" y1="33.02" x2="20.32" y2="38.1" width="0.1524" layer="91"/>
@@
 <pinref part="IC1" gate="G$1" pin="EN_3.3V"/>
 <wire x1="22.86" y1="33.02" x2="20.32" y2="33.02" width="0.1524" layer="91"/>
-<junction x="20.32" y="33.02"/>
 <wire x1="20.32" y1="38.1" x2="15.24" y2="38.1" width="0.1524" layer="91"/>
 <junction x="15.24" y="38.1"/>
@@
 <pinref part="C13" gate="G$1" pin="1"/>
 <pinref part="P+1" gate="G$1" pin="3.3V"/>
-<wire x1="55.88" y1="43.18" x2="55.88" y2="45.72" width="0.1524" layer="91"/>
+<wire x1="55.88" y1="30.48" x2="55.88" y2="33.02" width="0.1524" layer="91"/>
 <pinref part="IC1" gate="G$1" pin="3.3V"/>
-<wire x1="55.88" y1="45.72" x2="55.88" y2="48.26" width="0.1524" layer="91"/>
-<wire x1="48.26" y1="33.02" x2="50.8" y2="33.02" width="0.1524" layer="91"/>
-<wire x1="50.8" y1="33.02" x2="50.8" y2="45.72" width="0.1524" layer="91"/>
-<wire x1="50.8" y1="45.72" x2="55.88" y2="45.72" width="0.1524" layer="91"/>
-<junction x="55.88" y="45.72"/>
+<wire x1="55.88" y1="33.02" x2="55.88" y2="35.56" width="0.1524" layer="91"/>
+<wire x1="48.26" y1="33.02" x2="55.88" y2="33.02" width="0.1524" layer="91"/>
+<junction x="55.88" y="33.02"/>
 </segment>
 <segment>
@@
 </segment>
 </net>
-<net name="3.0V" class="0">
-<segment>
-<pinref part="C14" gate="G$1" pin="1"/>
-<pinref part="U$5" gate="G$1" pin="3.0V"/>
-<wire x1="55.88" y1="15.24" x2="55.88" y2="17.78" width="0.1524" layer="91"/>
-<pinref part="IC1" gate="G$1" pin="3.0"/>
-<wire x1="55.88" y1="17.78" x2="55.88" y2="20.32" width="0.1524" layer="91"/>
-<wire x1="48.26" y1="27.94" x2="50.8" y2="27.94" width="0.1524" layer="91"/>
-<wire x1="50.8" y1="27.94" x2="50.8" y2="17.78" width="0.1524" layer="91"/>
-<wire x1="50.8" y1="17.78" x2="55.88" y2="17.78" width="0.1524" layer="91"/>
-<junction x="55.88" y="17.78"/>
-</segment>
-</net>

Commit message: Renumber components for silk
Parts:
- IC1: value MIC5335-SPYMT -> TXB0108RGY; device biomimetic:MIC5335-SPYMT -> biomimetic:TXB0108RGY
- IC2: value TXB0108RGY -> MIC5335-SPYMT; device biomimetic:TXB0108RGY -> biomimetic:MIC5335-SPYMT
- JP3: value BATTERY -> CONSOLE; device biomimetic:JST-RCY-MALE-NOSILK -> biomimetic:M04MOLEX_5267
- JP5: value CONSOLE -> BATTERY; device biomimetic:M04MOLEX_5267 -> biomimetic:JST-RCY-MALE-NOSILK
- renumbered C10 to C101, C11 to C100, C12 to C4, C13 to C3, C15 to C1, C16 to C2
Connections:
- net 1.8V: now also IC1.OE, IC1.VCCA, JP3.1; no longer IC2.OE, IC2.VCCA, JP5.1
- net 3.3V: now also IC1.VCCB, IC2.3.3V; no longer IC1.3.3V, IC2.VCCB
- net GND: now also IC1.A1, IC1.A4, IC1.A5, IC1.A6, IC1.A7, IC1.A8, IC1.B1, IC1.B4, IC1.B5, IC1.B6, IC1.B7, IC1.B8, IC2.EN_3.0V, JP3.4, JP5.1; no longer IC1.EN_3.0V, IC2.A1, IC2.A4, IC2.A5, IC2.A6, IC2.A7, IC2.A8, IC2.B1, IC2.B4, IC2.B5, IC2.B6, IC2.B7, IC2.B8, JP3.1, JP5.4
- net IMAGEPROC_RXD: now also IC1.B2; no longer IC2.B2
- net IMAGEPROC_TXD: now also IC1.B3; no longer IC2.B3
- net ODROID_RXD: now also IC1.A3, JP3.3; no longer IC2.A3, JP5.3
- net ODROID_TXD: now also IC1.A2, JP3.2; no longer IC2.A2, JP5.2
- net V_BATT: now also IC2.EN_3.3V, IC2.VIN, JP5.2; no longer IC1.EN_3.3V, IC1.VIN, JP3.2
